File: Pro/PCB/Lily58_Pro.kicad_pcb (KiCad board)
At the start: 2 copper layers, 142.5 x 106.3 mm, 87 parts, among them J1 LED, J2 4PIN, J3 OLED, P1 i2c_pin, P2 i2c_pin, SW1 SW_PUSH, SW10 SW_PUSH, SW11 SW_PUSH, SW12 SW_PUSH, SW13 SW_PUSH, SW14 SW_PUSH, SW15 SW_PUSH, SW16 SW_PUSH, SW17 SW_PUSH, SW18 SW_PUSH, SW19 SW_PUSH, SW2 SW_PUSH, SW20 SW_PUSH, SW21 SW_PUSH, SW22 SW_PUSH, SW23 SW_PUSH, SW24 SW_PUSH, SW25 SW_PUSH, SW26 SW_PUSH, SW27 SW_PUSH, SW28 SW_PUSH, SW29 SW_PUSH, SW3 SW_PUSH, SW4 SW_PUSH, SW5 SW_PUSH, SW6 SW_PUSH, SW7 SW_PUSH, SW8 SW_PUSH, SW9 SW_PUSH, U1 ProMicro

Commit message: Wireless
Parts:
- removed G*** (x2): LOGO, Lily58-footprint:lily58_logo_2
- removed G*** (x2): LOGO, Lily58-footprint:lily58_logo_Pro
- added J4: Conn_01x02, Connector_PinSocket_2.54mm:PinSocket_1x02_P2.54mm_Vertical, F.Cu at (86.6, 76.2)
- added 卧式开关1: ~, switch:SW-TH_SK12D07VG5, F.Cu at (85.7, 96.5)
- JP1, JP2, JP3, JP4, JP5, JP6, JP7, JP8: value (none) -> Jumper_NO_Small
- U1: value ProMicro -> nice_nano; footprint Lily58-footprint:ProMicro_rev2 -> nice-nano-kicad:NiceNano_rev2
- moved U1 12.4 mm to (107.4, 66.6)
Connections:
- D1 pad 2: Net-(D1-Pad2) -> Net-(D1-A)
- D10 pad 2: Net-(D10-Pad2) -> Net-(D10-A)
- D11 pad 2: Net-(D11-Pad2) -> Net-(D11-A)
- D12 pad 2: Net-(D12-Pad2) -> Net-(D12-A)
- D13 pad 2: Net-(D13-Pad2) -> Net-(D13-A)
- D14 pad 2: Net-(D14-Pad2) -> Net-(D14-A)
- D15 pad 2: Net-(D15-Pad2) -> Net-(D15-A)
- D16 pad 2: Net-(D16-Pad2) -> Net-(D16-A)
- D17 pad 2: Net-(D17-Pad2) -> Net-(D17-A)
- D18 pad 2: Net-(D18-Pad2) -> Net-(D18-A)
- D19 pad 2: Net-(D19-Pad2) -> Net-(D19-A)
- D2 pad 2: Net-(D2-Pad2) -> Net-(D2-A)
- D20 pad 2: Net-(D20-Pad2) -> Net-(D20-A)
- D21 pad 2: Net-(D21-Pad2) -> Net-(D21-A)
- D22 pad 2: Net-(D22-Pad2) -> Net-(D22-A)
- D23 pad 2: Net-(D23-Pad2) -> Net-(D23-A)
- D24 pad 2: Net-(D24-Pad2) -> Net-(D24-A)
- D25 pad 2: Net-(D25-Pad2) -> Net-(D25-A)
- D26 pad 2: Net-(D26-Pad2) -> Net-(D26-A)
- D27 pad 2: Net-(D27-Pad2) -> Net-(D27-A)
- D28 pad 2: Net-(D28-Pad2) -> Net-(D28-A)
- D29 pad 2: Net-(D29-Pad2) -> Net-(D29-A)
- D3 pad 2: Net-(D3-Pad2) -> Net-(D3-A)
- D4 pad 2: Net-(D4-Pad2) -> Net-(D4-A)
- D5 pad 2: Net-(D5-Pad2) -> Net-(D5-A)
- D6 pad 2: Net-(D6-Pad2) -> Net-(D6-A)
- D7 pad 2: Net-(D7-Pad2) -> Net-(D7-A)
- D8 pad 2: Net-(D8-Pad2) -> Net-(D8-A)
- D9 pad 2: Net-(D9-Pad2) -> Net-(D9-A)
- U1 pad 1: LED -> Bnegative
- U1 pad 10: row2 -> row1
- U1 pad 11: row3 -> row2
- U1 pad 12: row4 -> row3
- U1 pad 13: col5 -> row4
- U1 pad 14: col4 -> col5
- U1 pad 15: col3 -> col4
- U1 pad 16: col2 -> col3
- U1 pad 17: col1 -> col2
- U1 pad 18: col0 -> col1
- U1 pad 19: Net-(U1-Pad19) -> col0
- U1 pad 2: DATA -> LED
- U1 pad 20: Net-(U1-Pad20) -> unconnected-(U1-AIN5/P0.29-Pad20)
- U1 pad 21: VCC -> unconnected-(U1-AIN7/P0.31-Pad21)
- U1 pad 22: RESET -> VCC
- U1 pad 23: GND -> RESET
- U1 pad 24: Net-(U1-Pad24) -> GND
- U1 pad 3: GND -> DATA
- U1 pad 5: SDA -> GND
- U1 pad 6: SCL -> SDA
- U1 pad 7: Net-(U1-Pad7) -> SCL
- U1 pad 8: row0 -> unconnected-(U1-P0.22-Pad8)
- U1 pad 9: row1 -> row0
Routing:
- net PowerIn: track 0.00 -> 85.9 mm
- net Bnegative: track 0.00 -> 64.8 mm, vias 0 -> 2
- net Bpositive: track 0.00 -> 20.5 mm
- net unconnected-(U1-P0.22-Pad8): track 0.00 -> 17.0 mm, vias 0 -> 1
- net Net-(U1-Pad7): track 17.0 -> 0.00 mm, vias 1 -> 0
- net unconnected-(U1-BATIN/P0.04-Pad25): track 0.00 -> 14.4 mm
- net unconnected-(U1-AIN7/P0.31-Pad21): track 0.00 -> 14.4 mm
- net unconnected-(U1-AIN5/P0.29-Pad20): track 0.00 -> 14.4 mm
- net Net-(U1-Pad24): track 14.4 -> 0.00 mm
- net Net-(U1-Pad20): track 14.4 -> 0.00 mm
- net Net-(U1-Pad19): track 14.4 -> 0.00 mm
- net col4: track 319.5 -> 317.2 mm
Other:
- board size 142.5 x 106.3 mm -> 143.2 x 106.3 mm
- net class Default removed
- net class GND removed
- net class VCC removed
